Commit message: missing hyqreal leg urdf

File: resources/urdfs/hyq/urdf/leg/hyq_leg_RF.urdf (robot description, URDF)
Before this commit: robot hyq, 5 links, 4 joints
Links:
- removed link foot
- added link rf_foot; collision sphere radius=0.032; visual sphere radius=0.032
- link rf_hipassembly: mass 2.93 -> 4.973275; geometry visual cylinder length=0.117 radius=0.0444
- link rf_lowerleg: mass 0.881 -> 1.291954; geometry collision mesh filename=package://hyqreal_description/meshes/leg/lowerleg_decimated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 scale=0.001 0.001 0.001; visual mesh filename=package://hyqreal_description/meshes/leg/lowerleg.dae scale=0.001 0.001 0.001
- link rf_upperleg: mass 2.638 -> 5.877927; geometry collision mesh filename=package://hyqreal_description/meshes/leg/upperleg.dae scale=0.001 0.001 0.001; visual mesh filename=package://hyqreal_description/meshes/leg/upperleg.dae scale=0.001 0.001 0.001
Joints:
- removed joint foot_joint
- added joint rf_foot_joint: type fixed, parent rf_lowerleg, child rf_foot, origin xyz=0.38 0 0 rpy=1.57079632679 0 -1.57079632679
- joint rf_haa_joint: axis 0.0 0.0 1.0 -> 0 0 1; limit lower=-1.2217304764 upper=0.436332312999 effort=150.0 velocity=12.0 -> lower=-0.733038285838 upper=0.401425727959 effort=173.0 velocity=12.0; origin xyz=0.3735 -0.207 0.0 rpy=0 1.57079632679 0 -> xyz=0.4435 -0.139 0 rpy=0 1.57079632679 0
- joint rf_hfe_joint: axis 0.0 0.0 1.0 -> 0 0 1; limit lower=-0.872664625997 upper=1.2217304764 effort=150.0 velocity=12.0 -> lower=-2.35619449019 upper=2.35619449019 effort=208 velocity=12.0; origin xyz=0.08 0.0 0.0 rpy=1.57079632679 0.0 0.0 -> xyz=0 -0.117 0 rpy=-1.57079632679 0 0
- joint rf_kfe_joint: axis 0.0 0.0 1.0 -> 0 0 1; limit lower=-2.44346095279 upper=-0.349065850399 effort=150.0 velocity=12.0 -> lower=-2.77001205584 upper=-0.669857366915 effort=249 velocity=12.0; origin xyz=0.35 0.0 0.0 rpy=0.0 0.0 0.0 -> xyz=0.36 0 0 rpy=0 0 0
